File: hardware/Jude_FlightController.kicad_sch (KiCad schematic)
At the start: 68 parts, among them J1 Servo, J2 Servo, J3 Servo, J4 Servo, J5 Servo, J6 Servo, SW1 TS-1088-AR02016, SW2 TS-1088-AR02016, U1 BMP580, U2 ICM-45686, U3 JBL-102010052, U4 LMR51430XFDDCR, U5 QMC5883P, U6 SAM-M10Q-00B, U8 STM32F722RET6TR, X1 Q13FC1350000400, X2 X322525MOB4SI

Commit message: added footprints and separated component groups in PCB
Parts:
- C23, C8: footprint Capacitor_SMD:C_01005_0402Metric -> Capacitor_SMD:C_0805_2012Metric
- Cout1: footprint Capacitor_SMD:C_0402_1005Metric -> Capacitor_SMD:C_0805_2012Metric
- Cout2: renamed from Cout; footprint Capacitor_SMD:C_0402_1005Metric -> Capacitor_SMD:C_0805_2012Metric
- J1, J2, J3, J4, J5, J6: footprint (none) -> Connector_PinHeader_2.54mm:PinHeader_1x03_P2.54mm_Vertical
- L1: footprint Inductor_SMD:L_01005_0402Metric -> easyeda2kicad:IND-SMD_L3.0-W3.0
- LED1: footprint easyeda2kicad:LED1206-R-RD_RED -> LED_SMD:LED_0402_1005Metric
- U8: footprint easyeda2kicad:LQFP-64_L10.0-W10.0-P0.50-LS12.0-BL -> Package_QFP:LQFP-64_10x10mm_P0.5mm
- renumbered Cboot to Cboot1, Cin to Cin1, I2CPullupSCL to I2CPullupSCL1, I2CPullupSDA to I2CPullupSDA1, Rfbb to Rfbb1, Rfbt to Rfbt1
Changed lines of the file:
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@@
 		)
 	)
-	(label ""
-		(at 41.91 54.61 0)
-		(effects
-			(font
-				(size 1.27 1.27)
-			)
-			(justify left bottom)
-		)
-	)
 	(label "LED_STATUS"
 		(at 323.85 57.15 0)
@@
 			)
 		)
-		(property "Footprint" ""
+		(property "Footprint" "Connector_PinHeader_2.54mm:PinHeader_1x03_P2.54mm_Vertical"
 			(at 167.64 274.32 0)
 			(hide yes)
@@
 			)
 		)
-		(property "Footprint" "Capacitor_SMD:C_0402_1005Metric"
+		(property "Footprint" "Capacitor_SMD:C_0805_2012Metric"
 			(at 96.2152 269.24 0)
 			(hide yes)
@@
 		(dnp no)
 		(fields_autoplaced yes)
-		(property "Reference" "I2CPullupSDA"
+		(property "Reference" "I2CPullupSDA1"
 			(at 255.27 120.6499 0)
 			(show_name no)
@@
 			(project "Jude_FlightController"
 				(path "/9932845b-f9a6-442a-bb24-38eb839f734b"
-					(reference "I2CPullupSDA")
+					(reference "I2CPullupSDA1")
 					(unit 1)
 				)
@@
 		(in_pos_files yes)
 		(dnp no)
-		(property "Reference" "Cin"
+		(property "Reference" "Cin1"
 			(at 26.416 256.794 0)
 			(show_name no)
@@
 			(project "Jude_FlightController"
 				(path "/9932845b-f9a6-442a-bb24-38eb839f734b"
-					(reference "Cin")
+					(reference "Cin1")
 					(unit 1)
 				)
@@
 			)
 		)
-		(property "Footprint" ""
+		(property "Footprint" "Connector_PinHeader_2.54mm:PinHeader_1x03_P2.54mm_Vertical"
 			(at 187.96 245.11 0)
 			(hide yes)
@@
 		(in_pos_files yes)
 		(dnp no)
-		(property "Reference" "Rfbt"
+		(property "Reference" "Rfbt1"
 			(at 79.756 261.62 0)
 			(show_name no)
@@
 			(project "Jude_FlightController"
 				(path "/9932845b-f9a6-442a-bb24-38eb839f734b"
-					(reference "Rfbt")
+					(reference "Rfbt1")
 					(unit 1)
 				)
@@
 			)
 		)
-		(property "Footprint" ""
+		(property "Footprint" "Connector_PinHeader_2.54mm:PinHeader_1x03_P2.54mm_Vertical"
 			(at 167.64 259.08 0)
 			(hide yes)
@@
 			)
 		)
-		(property "Footprint" ""
+		(property "Footprint" "Connector_PinHeader_2.54mm:PinHeader_1x03_P2.54mm_Vertical"
 			(at 167.64 245.11 0)
 			(hide yes)
@@
 		(in_pos_files yes)
 		(dnp no)
-		(property "Reference" "Cout"
+		(property "Reference" "Cout2"
 			(at 87.376 263.398 0)
 			(show_name no)
@@
 			)
 		)
-		(property "Footprint" "Capacitor_SMD:C_0402_1005Metric"
+		(property "Footprint" "Capacitor_SMD:C_0805_2012Metric"
 			(at 87.3252 269.24 0)
 			(hide yes)
@@
 			(project "Jude_FlightController"
 				(path "/9932845b-f9a6-442a-bb24-38eb839f734b"
-					(reference "Cout")
+					(reference "Cout2")
 					(unit 1)
 				)
@@
 			)
 		)
-		(property "Footprint" "easyeda2kicad:LQFP-64_L10.0-W10.0-P0.50-LS12.0-BL"
+		(property "Footprint" "Package_QFP:LQFP-64_10x10mm_P0.5mm"
 			(at 355.6 123.19 0)
 			(hide yes)
@@
 			)
 		)
-		(property "Footprint" ""
+		(property "Footprint" "Connector_PinHeader_2.54mm:PinHeader_1x03_P2.54mm_Vertical"
 			(at 187.96 259.08 0)
 			(hide yes)
@@
 			)
 		)
-		(property "Footprint" "Capacitor_SMD:C_01005_0402Metric"
+		(property "Footprint" "Capacitor_SMD:C_0805_2012Metric"
 			(at 277.8252 261.62 0)
 			(hide yes)
@@
 			)
 		)
-		(property "Footprint" "Capacitor_SMD:C_01005_0402Metric"
+		(property "Footprint" "Capacitor_SMD:C_0805_2012Metric"
 			(at 82.55 171.7548 0)
 			(hide yes)
@@
 		(dnp no)
 		(fields_autoplaced yes)
-		(property "Reference" "Rfbb"
+		(property "Reference" "Rfbb1"
 			(at 80.01 269.2399 0)
 			(show_name no)
@@
 			(project "Jude_FlightController"
 				(path "/9932845b-f9a6-442a-bb24-38eb839f734b"
-					(reference "Rfbb")
+					(reference "Rfbb1")
 					(unit 1)
 				)
@@
 			)
 		)
-		(property "Footprint" "easyeda2kicad:LED1206-R-RD_RED"
+		(property "Footprint" "LED_SMD:LED_0402_1005Metric"
 			(at 369.57 240.03 0)
 			(hide yes)
@@
 		(dnp no)
 		(fields_autoplaced yes)
-		(property "Reference" "I2CPullupSCL"
+		(property "Reference" "I2CPullupSCL1"
 			(at 255.27 110.4899 0)
 			(show_name no)
@@
 			(project "Jude_FlightController"
 				(path "/9932845b-f9a6-442a-bb24-38eb839f734b"
-					(reference "I2CPullupSCL")
+					(reference "I2CPullupSCL1")
 					(unit 1)
 				)
@@
 		(in_pos_files yes)
 		(dnp no)
-		(property "Reference" "Cboot"
+		(property "Reference" "Cboot1"
 			(at 65.786 250.698 0)
 			(show_name no)
@@
 			(project "Jude_FlightController"
 				(path "/9932845b-f9a6-442a-bb24-38eb839f734b"
-					(reference "Cboot")
+					(reference "Cboot1")
 					(unit 1)
 				)
@@
 			)
 		)
-		(property "Footprint" "Inductor_SMD:L_01005_0402Metric"
+		(property "Footprint" "easyeda2kicad:IND-SMD_L3.0-W3.0"
 			(at 72.39 257.81 0)
 			(hide yes)
@@
 			)
 		)
-		(property "Footprint" ""
+		(property "Footprint" "Connector_PinHeader_2.54mm:PinHeader_1x03_P2.54mm_Vertical"
 			(at 187.96 274.32 0)
 			(hide yes)
